Commit message: 🔧 Increased cable connector collision sphere size

File: ur_onrobot_description/urdf/ur_onrobot_macro.xacro (robot description, xacro)
@@ -54,5 +54,5 @@
                 <collision>
                 <geometry>
-                    <sphere radius="0.02"/>
+                    <sphere radius="0.03"/>
                 </geometry>
                 <origin xyz="0 0 0" rpy="0 0 0"/>
@@ -67,5 +67,5 @@
                 <collision>
                 <geometry>
-                    <sphere radius="0.02"/>
+                    <sphere radius="0.03"/>
                 </geometry>
                 <origin xyz="0 0 0" rpy="0 0 0"/>
